Commit message: rgb camera

File: src/arduinobot_description/urdf/arduinobot.urdf.xacro (robot description, xacro)
@@ -111,3 +111,18 @@
         <mimic joint="joint_4" multiplier="-1"/>
     </joint>
+    <link name="rgb_camera">
+        <visual>
+            <!-- <origin rpy="0 -0.5 1.57" xyz="0 0.45 0.2" /> -->
+            <origin rpy="-1.57 0 -1.57" xyz="-0.1 0.125 0.15"/>
+            <geometry>
+                <mesh filename="package://arduinobot_description/meshes/pi_camera.STL" scale="0.01 0.01 0.01" />
+            </geometry>
+        </visual>
+    </link>
+    <joint name="rgb_camera_joint" type="fixed">
+        <parent link="base_link" />
+        <child link="rgb_camera" />
+        <!-- <origin rpy="0 0 0" xyz="0 0 0" /> -->
+        <origin xyz="0 0.45 0.2" rpy="0 -0.5 1.57"/>
+    </joint>
 </robot>

Commit message: gazebo!

File: src/arduinobot_description/urdf/arduinobot.urdf.xacro (robot description, xacro)
@@ -4,6 +4,17 @@
     <xacro:property name="effort" value="30.0" />
     <xacro:property name="velocity" value="10.0" />
+    <xacro:macro name="default_inertial" params="mass">
+        <inertial>
+            <mass value="${mass}" />
+            <inertia
+                ixx="1.0" ixy="0.0" ixz="0.0"
+                iyy="1.0" iyz="0.0"
+                izz="1.0"
+            />
+        </inertial>
+    </xacro:macro>
     <link name="world" />
     <link name="base_link">
+        <xacro:default_inertial mass="1.0" />
         <visual>
             <origin rpy="0 0 0" xyz="-0.5 -0.5 0" />
@@ -12,4 +23,10 @@
             </geometry>
         </visual>
+        <collision>
+            <origin rpy="0 0 0" xyz="-0.5 -0.5 0" />
+            <geometry>
+                <mesh filename="package://arduinobot_description/meshes/basement.STL" scale="0.01 0.01 0.01" />
+            </geometry>
+        </collision>
     </link>
     <joint name="virtual_joint" type="fixed">
@@ -19,4 +36,5 @@
     </joint>
     <link name="base_plate">
+        <xacro:default_inertial mass="0.1" />
         <visual>
             <origin rpy="0 0 0" xyz="-0.39 -0.39 -0.56" />
@@ -25,4 +43,10 @@
             </geometry>
         </visual>
+        <collision>
+            <origin rpy="0 0 0" xyz="-0.39 -0.39 -0.56" />
+            <geometry>
+                <mesh filename="package://arduinobot_description/meshes/base_plate.STL" scale="0.01 0.01 0.01" />
+            </geometry>
+        </collision>
     </link>
     <joint name="joint_1" type="revolute">
@@ -34,4 +58,5 @@
     </joint>
     <link name="forward_drive_arm">
+        <xacro:default_inertial mass="0.1" />
         <visual>
             <origin rpy=" 0 -${PI / 2} ${PI / 2}" xyz="0.19 0.06 -0.08"/>
@@ -40,4 +65,10 @@
             </geometry>
         </visual>
+        <collision>
+            <origin rpy=" 0 -${PI / 2} ${PI / 2}" xyz="0.19 0.06 -0.08"/>
+            <geometry>
+                <mesh filename="package://arduinobot_description/meshes/forward_drive_arm.STL" scale="0.01 0.01 0.01"/>
+            </geometry>
+        </collision>
     </link>
   <joint name ="joint_2" type="revolute">
@@ -50,4 +81,5 @@
     </joint>
     <link name="horizontal_arm">
+        <xacro:default_inertial mass="0.1" />
         <visual>
             <origin rpy="${PI / 2} 0 ${PI / 2}" xyz="-0.03 -0.4 -0.06"/>
@@ -56,4 +88,10 @@
             </geometry>
         </visual>
+        <collision>
+            <origin rpy="${PI / 2} 0 ${PI / 2}" xyz="-0.03 -0.4 -0.06"/>
+            <geometry>
+                <mesh filename="package://arduinobot_description/meshes/horizontal_arm.STL" scale="0.01 0.01 0.01"/>
+            </geometry>
+        </collision>
     </link>
     <joint name ="joint_3" type="revolute">
@@ -66,4 +104,5 @@
     </joint>
     <link name="claw_support">
+        <xacro:default_inertial mass="0.05" />
         <visual>
             <origin rpy="0 0 ${PI / 2}" xyz="0 -0.05 -0.15"/>
@@ -72,4 +111,10 @@
             </geometry>
         </visual>
+        <collision>
+            <origin rpy="0 0 ${PI / 2}" xyz="0 -0.05 -0.15"/>
+            <geometry>
+                <mesh filename="package://arduinobot_description/meshes/claw_support.STL" scale="0.01 0.01 0.01"/>
+            </geometry>
+        </collision>
     </link>
     <joint name ="horizontal_arm_to_claw_support" type="fixed">
@@ -79,4 +124,5 @@
     </joint>
     <link name="gripper_right">
+        <xacro:default_inertial mass="0.01" />
         <visual>
             <origin rpy="0 0 -${PI / 2}" xyz="-0.1 0.50 -0.1"/>
@@ -85,6 +131,13 @@
             </geometry>
         </visual>
+        <collision>
+            <origin rpy="0 0 -${PI / 2}" xyz="-0.1 0.50 -0.1"/>
+            <geometry>
+                <mesh filename="package://arduinobot_description/meshes/right_finger.STL" scale="0.01 0.01 0.01"/>
+            </geometry>
+        </collision>
     </link>
     <link name="gripper_left">
+        <xacro:default_inertial mass="0.01" />
         <visual>
             <origin rpy="0 0 -${PI / 2}" xyz="-0.04 0.50 -0.1"/>
@@ -93,4 +146,10 @@
             </geometry>
         </visual>
+        <collision>
+            <origin rpy="0 0 -${PI / 2}" xyz="-0.04 0.50 -0.1"/>
+            <geometry>
+                <mesh filename="package://arduinobot_description/meshes/left_finger.STL" scale="0.01 0.01 0.01"/>
+            </geometry>
+        </collision>
     </link>
     <joint name ="joint_4" type="revolute">
@@ -119,4 +178,10 @@
             </geometry>
         </visual>
+        <collision>
+            <origin rpy="-1.57 0 -1.57" xyz="-0.1 0.125 0.15"/>
+            <geometry>
+                <mesh filename="package://arduinobot_description/meshes/pi_camera.STL" scale="0.01 0.01 0.01" />
+            </geometry>
+        </collision>
     </link>
     <joint name="rgb_camera_joint" type="fixed">

Commit message: section 4 - copied over
copied over from github repo
working in gazebo with fixed arm

File: src/arduinobot_description/urdf/arduinobot.urdf.xacro (robot description, xacro)
@@ -1,65 +1,58 @@
 <?xml version="1.0"?>
 <robot xmlns:xacro="http://www.ros.org/wiki/xacro" name="arduinobot">
-    <xacro:arg name="is_ignition" default="true" doc="Set to true if using Ignition Gazebo, false for Gazebo Classic." />
+    <!-- Start GZ or Ignition depending on ROS 2 Version -->
+    <xacro:arg name="is_ignition" default="true"/>
+    <!-- Include Gazebo Parameters -->
     <xacro:include filename="$(find arduinobot_description)/urdf/arduinobot_gazebo.xacro" />
+    <!-- Include ros2_control Plugins -->
     <xacro:include filename="$(find arduinobot_description)/urdf/arduinobot_ros2_control.xacro" />
-    <xacro:property name="PI" value="3.14159" />
+    <!-- Useful XACRO Variables (Properties) -->
+    <xacro:property name="PI" value="3.14159265359" />
     <xacro:property name="effort" value="30.0" />
     <xacro:property name="velocity" value="10.0" />
+    <!-- Useful Macros -->
     <xacro:macro name="default_inertial" params="mass">
         <inertial>
+            <origin xyz="0 0 0" rpy="0 0 0"/>
             <mass value="${mass}" />
-            <inertia
-                ixx="1.0" ixy="0.0" ixz="0.0"
-                iyy="1.0" iyz="0.0"
-                izz="1.0"
-            />
+            <inertia ixx="1.0" ixy="0.0" ixz="0.0"
+                     iyy="1.0" iyz="0.0"
+                     izz="1.0" />
         </inertial>
     </xacro:macro>
-    <link name="world" />
+    <!-- Links -->
+    <link name="world"/>
     <link name="base_link">
-        <xacro:default_inertial mass="1.0" />
+        <xacro:default_inertial mass="1.0"/>
         <visual>
-            <origin rpy="0 0 0" xyz="-0.5 -0.5 0" />
+            <origin rpy="0 0 0" xyz="-0.5 -0.5 0"/>
             <geometry>
-                <mesh filename="package://arduinobot_description/meshes/basement.STL" scale="0.01 0.01 0.01" />
+                <mesh filename="package://arduinobot_description/meshes/basement.STL" scale="0.01 0.01 0.01"/>
             </geometry>
         </visual>
         <collision>
-            <origin rpy="0 0 0" xyz="-0.5 -0.5 0" />
+            <origin rpy="0 0 0" xyz="-0.5 -0.5 0"/>
             <geometry>
-                <mesh filename="package://arduinobot_description/meshes/basement.STL" scale="0.01 0.01 0.01" />
+                <mesh filename="package://arduinobot_description/meshes/basement.STL" scale="0.01 0.01 0.01"/>
             </geometry>
         </collision>
     </link>
-    <joint name="virtual_joint" type="fixed">
-        <parent link="world" />
-        <child link="base_link" />
-        <origin rpy="0 0 0" xyz="0 0 0" />
-    </joint>
     <link name="base_plate">
-        <xacro:default_inertial mass="0.1" />
+        <xacro:default_inertial mass="0.1"/>
         <visual>
-            <origin rpy="0 0 0" xyz="-0.39 -0.39 -0.56" />
+            <origin rpy="0 0 0" xyz="-0.39 -0.39 -0.56"/>
             <geometry>
-                <mesh filename="package://arduinobot_description/meshes/base_plate.STL" scale="0.01 0.01 0.01" />
+                <mesh filename="package://arduinobot_description/meshes/base_plate.STL" scale="0.01 0.01 0.01"/>
             </geometry>
         </visual>
         <collision>
-            <origin rpy="0 0 0" xyz="-0.39 -0.39 -0.56" />
+            <origin rpy="0 0 0" xyz="-0.39 -0.39 -0.56"/>
             <geometry>
-                <mesh filename="package://arduinobot_description/meshes/base_plate.STL" scale="0.01 0.01 0.01" />
+                <mesh filename="package://arduinobot_description/meshes/base_plate.STL" scale="0.01 0.01 0.01"/>
             </geometry>
         </collision>
     </link>
-    <joint name="joint_1" type="revolute">
-        <parent link="base_link" />
-        <child link="base_plate" />
-        <axis xyz="0 0 1" />
-        <origin rpy="0 0 0" xyz="0 0 0.307" />
-        <limit upper="-${PI/2}" lower="${PI/2}" effort="${effort}" velocity="${velocity}" />
-    </joint>
     <link name="forward_drive_arm">
-        <xacro:default_inertial mass="0.1" />
+        <xacro:default_inertial mass="0.1"/>
         <visual>
             <origin rpy=" 0 -${PI / 2} ${PI / 2}" xyz="0.19 0.06 -0.08"/>
@@ -75,14 +68,6 @@
         </collision>
     </link>
-  <joint name ="joint_2" type="revolute">
-        <parent link="base_plate"/>
-        <child link = "forward_drive_arm"/>
-        <origin xyz="-0.02 0 0.35"/>
-        <axis xyz="1 0 0"/>
-        <limit lower="-${PI / 2}" upper="${PI / 2}"
-                effort="${effort}" velocity="${velocity}"/>
-    </joint>
     <link name="horizontal_arm">
-        <xacro:default_inertial mass="0.1" />
+        <xacro:default_inertial mass="0.1"/>
         <visual>
             <origin rpy="${PI / 2} 0 ${PI / 2}" xyz="-0.03 -0.4 -0.06"/>
@@ -98,14 +83,6 @@
         </collision>
     </link>
-    <joint name ="joint_3" type="revolute">
-        <parent link="forward_drive_arm"/>
-        <child link = "horizontal_arm"/>
-        <origin xyz="0 0 0.8"/>
-        <axis xyz="1 0 0"/>
-        <limit lower="-${PI / 2}" upper="${PI / 2}"
-               effort="${effort}" velocity="${velocity}"/>
-    </joint>
     <link name="claw_support">
-        <xacro:default_inertial mass="0.05" />
+        <xacro:default_inertial mass="0.05"/>
         <visual>
             <origin rpy="0 0 ${PI / 2}" xyz="0 -0.05 -0.15"/>
@@ -121,11 +98,6 @@
         </collision>
     </link>
-    <joint name ="horizontal_arm_to_claw_support" type="fixed">
-        <parent link="horizontal_arm"/>
-        <child link = "claw_support"/>
-        <origin xyz="0 0.82 0"/>
-    </joint>
     <link name="gripper_right">
-        <xacro:default_inertial mass="0.01" />
+        <xacro:default_inertial mass="0.01"/>
         <visual>
             <origin rpy="0 0 -${PI / 2}" xyz="-0.1 0.50 -0.1"/>
@@ -142,5 +114,5 @@
     </link>
     <link name="gripper_left">
-        <xacro:default_inertial mass="0.01" />
+        <xacro:default_inertial mass="0.01"/>
         <visual>
             <origin rpy="0 0 -${PI / 2}" xyz="-0.04 0.50 -0.1"/>
@@ -156,4 +128,39 @@
         </collision>
     </link>
+    <!-- Joints -->
+    <joint name="virtual_joint" type="fixed">
+        <parent link="world"/>
+        <child link="base_link"/>
+        <origin xyz="0 0 0" rpy="0 0 0"/>
+    </joint>
+    <joint name ="joint_1" type="revolute">
+        <parent link="base_link"/>
+        <child link = "base_plate"/>
+        <origin xyz="0 0 0.307"/>
+        <axis xyz="0 0 1"/>
+        <limit lower="-${PI / 2}" upper="${PI / 2}"
+               effort="${effort}" velocity="${velocity}"/>
+    </joint>
+    <joint name ="joint_2" type="revolute">
+        <parent link="base_plate"/>
+        <child link = "forward_drive_arm"/>
+        <origin xyz="-0.02 0 0.35"/>
+        <axis xyz="1 0 0"/>
+        <limit lower="-${PI / 2}" upper="${PI / 2}"
+                effort="${effort}" velocity="${velocity}"/>
+    </joint>
+    <joint name ="joint_3" type="revolute">
+        <parent link="forward_drive_arm"/>
+        <child link = "horizontal_arm"/>
+        <origin xyz="0 0 0.8"/>
+        <axis xyz="1 0 0"/>
+        <limit lower="-${PI / 2}" upper="${PI / 2}"
+               effort="${effort}" velocity="${velocity}"/>
+    </joint>
+    <joint name ="horizontal_arm_to_claw_support" type="fixed">
+        <parent link="horizontal_arm"/>
+        <child link = "claw_support"/>
+        <origin xyz="0 0.82 0"/>
+    </joint>
     <joint name ="joint_4" type="revolute">
         <parent link="claw_support"/>
@@ -173,25 +180,3 @@
         <mimic joint="joint_4" multiplier="-1"/>
     </joint>
-    <link name="rgb_camera">
-        <xacro:default_inertial mass="0.001" />
-        <visual>
-            <!-- <origin rpy="0 -0.5 1.57" xyz="0 0.45 0.2" /> -->
-            <origin rpy="-1.57 0 -1.57" xyz="-0.1 0.125 0.15"/>
-            <geometry>
-                <mesh filename="package://arduinobot_description/meshes/pi_camera.STL" scale="0.01 0.01 0.01" />
-            </geometry>
-        </visual>
-        <collision>
-            <origin rpy="-1.57 0 -1.57" xyz="-0.1 0.125 0.15"/>
-            <geometry>
-                <mesh filename="package://arduinobot_description/meshes/pi_camera.STL" scale="0.01 0.01 0.01" />
-            </geometry>
-        </collision>
-    </link>
-    <joint name="rgb_camera_joint" type="fixed">
-        <parent link="base_link" />
-        <child link="rgb_camera" />
-        <!-- <origin rpy="0 0 0" xyz="0 0 0" /> -->
-        <origin xyz="0 0.45 0.2" rpy="0 -0.5 1.57"/>
-    </joint>
 </robot>

File: src/arduinobot_description/urdf/arduinobot_gazebo.xacro (robot description, xacro)
@@ -1,11 +1,14 @@
 <?xml version="1.0"?>
 <robot xmlns:xacro="http://www.ros.org/wiki/xacro" name="arduinobot">
+  <!-- ROS 2 Control -->
   <gazebo>
-    <xacro:if value="${arg is_ignition}">
+    <!-- ROS 2 Humble -->
+    <xacro:if value="$(arg is_ignition)">
       <plugin filename="ign_ros2_control-system" name="ign_ros2_control::IgnitionROS2ControlPlugin">
         <parameters>$(find arduinobot_controller)/config/arduinobot_controllers.yaml</parameters>
       </plugin>
-      </xacro:if>
-    <xacro:unless value="${arg is_ignition}">
+    </xacro:if>
+    <!-- ROS 2 Iron or above -->
+    <xacro:unless value="$(arg is_ignition)">
       <plugin filename="gz_ros2_control-system" name="gz_ros2_control::GazeboSimROS2ControlPlugin">
         <parameters>$(find arduinobot_controller)/config/arduinobot_controllers.yaml</parameters>

File: src/arduinobot_description/urdf/arduinobot_ros2_control.xacro (robot description, xacro)
@@ -1,48 +1,51 @@
 <?xml version="1.0"?>
 <robot xmlns:xacro="http://www.ros.org/wiki/xacro" name="arduinobot">
-  <xacro:property name="PI" value="3.14159" />
-  <ros2_control type="system" name="RobotSystem">
-    <xacro:if value="$(arg is_ignition)">
-      <hardware>
-        <plugin>ign_ros2_control/IgnitionSystem</plugin>
-      </hardware>
-    </xacro:if>
-    <xacro:unless value="$(arg is_ignition)">
-      <hardware>
-        <plugin>gz_ros2_control/GazeboSimSystem</plugin>
-      </hardware>
-    </xacro:unless>
-    <joint name="joint_1">
-      <command_interface name="position">
-        <param name="min">-${PI/2}</param>
-        <param name="max">${PI/2}</param>
-      </command_interface>
-      <state_interface name="position" />
-    </joint>
-    <joint name="joint_2">
-      <command_interface name="position">
-        <param name="min">-${PI/2}</param>
-        <param name="max">${PI/2}</param>
-      </command_interface>
-      <state_interface name="position" />
-    </joint>
-    <joint name="joint_3">
-      <command_interface name="position">
-        <param name="min">-${PI/2}</param>
-        <param name="max">${PI/2}</param>
-      </command_interface>
-      <state_interface name="position" />
-    </joint>
-    <joint name="joint_4">
-      <command_interface name="position">
-        <param name="min">-${PI/2}</param>
-        <param name="max">0.0</param>
-      </command_interface>
-      <state_interface name="position" />
-    </joint>
-    <joint name="joint_5">
-      <param name="mimic">joint_4</param>
-      <param name="multiplier">-1</param>
-    </joint>
-  </ros2_control>
+    <ros2_control name="RobotSystem" type="system">
+        <xacro:property name="PI" value="3.14159265359" />
+        <!-- ros2_control Gazebo -->
+        <!-- ROS 2 Humble -->
+        <xacro:if value="$(arg is_ignition)">
+            <hardware>
+                <plugin>ign_ros2_control/IgnitionSystem</plugin>
+            </hardware>
+        </xacro:if>
+        <!-- ROS 2 Iron or above -->
+        <xacro:unless value="$(arg is_ignition)">
+            <hardware>
+                <plugin>gz_ros2_control/GazeboSimSystem</plugin>
+            </hardware>
+        </xacro:unless>
+        <joint name="joint_1">
+            <command_interface name="position">
+            <param name="min">-${PI / 2}</param>
+            <param name="max">${PI / 2}</param>
+            </command_interface>
+            <state_interface name="position"/>
+        </joint>
+        <joint name="joint_2">
+            <command_interface name="position">
+            <param name="min">-${PI / 2}</param>
+            <param name="max">${PI / 2}</param>
+            </command_interface>
+            <state_interface name="position"/>
+        </joint>
+        <joint name="joint_3">
+            <command_interface name="position">
+            <param name="min">-${PI / 2}</param>
+            <param name="max">${PI / 2}</param>
+            </command_interface>
+            <state_interface name="position"/>
+        </joint>
+        <joint name="joint_4">
+            <command_interface name="position">
+            <param name="min">-${PI / 2}</param>
+            <param name="max">0.0</param>
+            </command_interface>
+            <state_interface name="position"/>
+        </joint>
+        <joint name="joint_5">
+            <param name="mimic">joint_4</param>
+            <param name="multiplier">-1</param>
+        </joint>
+    </ros2_control>
 </robot>
